Commit message: perception_1

File: Ensamble_URDF_manipulator/urdf/Ensamble_URDF_2ndT.urdf (robot description, URDF)
Before this commit: robot robot, 10 links, 9 joints
Links:
- added link optical
- added link rgbd_cam, mass 0.1; visual box size=0.01 0.01 0.01
Joints:
- added joint optical_joint: type fixed, parent rgbd_cam, child optical, origin xyz=0.0 0.0 0.0 rpy=-1.5708 0.0 -1.5708
- added joint rgbd_link: type fixed, parent base_link_Chasis, child rgbd_cam, origin xyz=0.221 0.0 0.045 rpy=0.0 0.0 0.0

Commit message: integracion1

File: Ensamble_URDF_manipulator/urdf/Ensamble_URDF_2ndT.urdf (robot description, URDF)
Before this commit: robot robot, 12 links, 11 joints
Links:
- removed link Link_1_1_wheel
- removed link Link_1_2_wheel
- removed link Link_1_3_wheel
- removed link Link_1_4_wheel
- added link front_left_wheel, mass 0.622419475189309; collision mesh filename=package://Ensamble_URDF_2ndT/meshes/Link_1_4_wheel.STL; visual mesh filename=package://Ensamble_URDF_2ndT/meshes/Link_1_4_wheel.STL
- added link front_right_wheel, mass 0.622419475189309; collision mesh filename=package://Ensamble_URDF_2ndT/meshes/Link_1_3_wheel.STL; visual mesh filename=package://Ensamble_URDF_2ndT/meshes/Link_1_3_wheel.STL
- added link rear_left_wheel, mass 0.622419475189309; collision mesh filename=package://Ensamble_URDF_2ndT/meshes/Link_1_2_wheel.STL; visual mesh filename=package://Ensamble_URDF_2ndT/meshes/Link_1_2_wheel.STL
- added link rear_right_wheel, mass 0.622419475189312; collision mesh filename=package://Ensamble_URDF_2ndT/meshes/Link_1_1_wheel.STL; visual mesh filename=package://Ensamble_URDF_2ndT/meshes/Link_1_1_wheel.STL
- link base_link_Chasis: mass 5.34447797641956 -> 5.1498884920758
Joints:
- removed joint joint_1_1_wheel
- removed joint joint_1_2_wheel
- removed joint joint_1_3_wheel
- removed joint joint_1_4_wheel
- added joint joint_front_left: type continuous, parent base_link_Chasis, child front_left_wheel, origin xyz=0.08 0.19608 0.0195 rpy=-1.5708 0 0, axis 0 0 1
- added joint joint_front_right: type continuous, parent base_link_Chasis, child front_right_wheel, origin xyz=0.08 -0.19478 0.0195 rpy=1.5708 0 0, axis 0 0 -1
- added joint joint_rear_left: type continuous, parent base_link_Chasis, child rear_left_wheel, origin xyz=-0.12 0.19608 0.0195 rpy=-1.5708 0 0, axis 0 0 1
- added joint joint_rear_right: type continuous, parent base_link_Chasis, child rear_right_wheel, origin xyz=-0.12 -0.19478 0.0195 rpy=1.5708 0 0, axis 0 0 -1
