Commit message: Workin position controller

File: Ensamble_URDF_2ndT/urdf/Ensamble_URDF_2ndT.urdf (robot description, URDF)
Before this commit: robot robot, 10 links, 9 joints
Joints:
- joint joint_2_Arm: limit lower=-3.14 upper=3.14 effort=0 velocity=0 -> lower=-3.14 upper=3.14 effort=100 velocity=100
- joint joint_3_Arm: limit lower=-0.6 upper=1.4 effort=0 velocity=0 -> lower=-0.6 upper=1.4 effort=100 velocity=100
- joint joint_4_Arm: limit lower=-1.57 upper=1.2 effort=0 velocity=0 -> lower=-1.57 upper=1.2 effort=100 velocity=100
- joint joint_5_Arm: limit lower=-2.8 upper=2.8 effort=0 velocity=0 -> lower=-2.8 upper=2.8 effort=100 velocity=100

Commit message: Manipulator-mobile integration

File: Ensamble_URDF_2ndT/urdf/Ensamble_URDF_2ndT.urdf (robot description, URDF)
Before this commit: robot robot, 10 links, 9 joints
Links:
- removed link Link_1_1_wheel
- removed link Link_1_2_wheel
- removed link Link_1_3_wheel
- removed link Link_1_4_wheel
- added link front_left_wheel, mass 0.622419475189309; collision mesh filename=package://ensamble_mobile/meshes/Link_1_4_wheel.STL; visual mesh filename=package://ensamble_mobile/meshes/Link_1_4_wheel.STL
- added link front_right_wheel, mass 0.622419475189309; collision mesh filename=package://ensamble_mobile/meshes/Link_1_3_wheel.STL; visual mesh filename=package://ensamble_mobile/meshes/Link_1_3_wheel.STL
- added link optical
- added link rear_left_wheel, mass 0.622419475189309; collision mesh filename=package://ensamble_mobile/meshes/Link_1_2_wheel.STL; visual mesh filename=package://ensamble_mobile/meshes/Link_1_2_wheel.STL
- added link rear_right_wheel, mass 0.622419475189312; collision mesh filename=package://ensamble_mobile/meshes/Link_1_1_wheel.STL; visual mesh filename=package://ensamble_mobile/meshes/Link_1_1_wheel.STL
- added link rgbd_cam, mass 0.1; visual box size=0.01 0.01 0.01
- link base_link_Chasis: mass 5.34447797641956 -> 15.1498884920758; geometry collision mesh filename=package://ensamble_mobile/meshes/base_link_Chasis.STL; visual mesh filename=package://ensamble_mobile/meshes/base_link_Chasis.STL
Joints:
- removed joint joint_1_1_wheel
- removed joint joint_1_2_wheel
- removed joint joint_1_3_wheel
- removed joint joint_1_4_wheel
- added joint joint_front_left: type continuous, parent base_link_Chasis, child front_left_wheel, origin xyz=0.08 0.19608 0.0195 rpy=-1.5708 0 0, axis 0 0 1
- added joint joint_front_right: type continuous, parent base_link_Chasis, child front_right_wheel, origin xyz=0.08 -0.19478 0.0195 rpy=1.5708 0 0, axis 0 0 -1
- added joint joint_rear_left: type continuous, parent base_link_Chasis, child rear_left_wheel, origin xyz=-0.12 0.19608 0.0195 rpy=-1.5708 0 0, axis 0 0 1
- added joint joint_rear_right: type continuous, parent base_link_Chasis, child rear_right_wheel, origin xyz=-0.12 -0.19478 0.0195 rpy=1.5708 0 0, axis 0 0 -1
- added joint optical_joint: type fixed, parent rgbd_cam, child optical, origin xyz=0.0 0.0 0.0 rpy=-1.5708 0.0 -1.5708
- added joint rgbd_link: type fixed, parent base_link_Chasis, child rgbd_cam, origin xyz=0.221 0.0 0.045 rpy=0.0 0.0 0.0

File: mobile/ensamble_mobile/urdf/mobile.urdf (robot description, URDF)
Before this commit: robot robot, 7 links, 6 joints
Links:
- added link Link_2_Arm, mass 0.628890750175801; collision mesh filename=package://Ensamble_URDF_2ndT/meshes/Link_2_Arm.STL; visual mesh filename=package://Ensamble_URDF_2ndT/meshes/Link_2_Arm.STL
- added link Link_3_Arm, mass 0.253359108687758; collision mesh filename=package://Ensamble_URDF_2ndT/meshes/Link_3_Arm.STL; visual mesh filename=package://Ensamble_URDF_2ndT/meshes/Link_3_Arm.STL
- added link Link_4_Arm, mass 0.5315; collision mesh filename=package://Ensamble_URDF_2ndT/meshes/Link_4_Arm.STL; visual mesh filename=package://Ensamble_URDF_2ndT/meshes/Link_4_Arm.STL
- added link Link_5_Arm, mass 0.34582; collision mesh filename=package://Ensamble_URDF_2ndT/meshes/Link_5_Arm.STL; visual mesh filename=package://Ensamble_URDF_2ndT/meshes/Link_5_Arm.STL
- added link optical
- link base_link_Chasis: mass 5.1498884920758 -> 15.1498884920758
Joints:
- added joint joint_2_Arm: type revolute, parent base_link_Chasis, child Link_2_Arm, origin xyz=0 0 0.098503 rpy=0 0 0, axis 0 0 1, limit lower=-3.14 upper=3.14 effort=100 velocity=100
- added joint joint_3_Arm: type revolute, parent Link_2_Arm, child Link_3_Arm, origin xyz=0.063383 0.0021739 0.12369 rpy=1.5708 0 0, axis 0.034278 0 0.99941, limit lower=-0.6 upper=1.4 effort=100 velocity=100
- added joint joint_4_Arm: type revolute, parent Link_3_Arm, child Link_4_Arm, origin xyz=0.060241 0.1907 -0.0020662 rpy=0 0 0, axis -0.034278 0 -0.99941, limit lower=-1.57 upper=1.2 effort=100 velocity=100
- added joint joint_5_Arm: type revolute, parent Link_4_Arm, child Link_5_Arm, origin xyz=0.21278 -0.0095961 -0.0037813 rpy=0 0 0, axis -0.034278 0 -0.99941, limit lower=-2.8 upper=2.8 effort=100 velocity=100
- added joint optical_joint: type fixed, parent rgbd_cam, child optical, origin xyz=0.0 0.0 0.0 rpy=-1.5708 0.0 -1.5708
- joint rgbd_link: origin xyz=0.0221 0.0 0.0045 rpy=0.0 0.0 0.0 -> xyz=0.221 0.0 0.045 rpy=0.0 0.0 0.0

Commit message: Planner

File: Ensamble_URDF_2ndT/urdf/Ensamble_URDF_2ndT.urdf (robot description, URDF)
Before this commit: robot robot, 12 links, 11 joints
Joints:
- joint joint_3_Arm: limit lower=-0.6 upper=1.4 effort=100 velocity=100 -> lower=-10.6 upper=10.4 effort=100 velocity=100
- joint joint_4_Arm: limit lower=-1.57 upper=1.2 effort=100 velocity=100 -> lower=-10.57 upper=10.2 effort=100 velocity=100
- joint joint_5_Arm: limit lower=-2.8 upper=2.8 effort=100 velocity=100 -> lower=-20.8 upper=20.8 effort=100 velocity=100

Commit message: arm_position_actionlib

File: Ensamble_URDF_2ndT/urdf/Ensamble_URDF_2ndT.urdf (robot description, URDF)
Before this commit: robot robot, 12 links, 11 joints
Joints:
- joint joint_3_Arm: limit lower=-10.6 upper=10.4 effort=100 velocity=100 -> lower=-1.6 upper=1.4 effort=100 velocity=100
- joint joint_4_Arm: limit lower=-10.57 upper=10.2 effort=100 velocity=100 -> lower=-1.87 upper=1.2 effort=100 velocity=100
- joint joint_5_Arm: limit lower=-20.8 upper=20.8 effort=100 velocity=100 -> lower=-2.5 upper=2.5 effort=100 velocity=100

Commit message: integrated_urdf

File: Ensamble_URDF_2ndT/urdf/Ensamble_URDF_2ndT.urdf (robot description, URDF)
Before this commit: robot robot, 12 links, 11 joints
Links:
- removed link base_link_Chasis
- added link base_link, mass 15.1498884920758; collision mesh filename=package://ensamble_mobile/meshes/base_link_Chasis.STL; visual mesh filename=package://ensamble_mobile/meshes/base_link_Chasis.STL
- added link imu_link
Joints:
- added joint imu_joint: type fixed, parent base_link, child imu_link, origin xyz=0.221 0.0 0.045 rpy=0.0 0.0 0.0
- joint dummy_joint: child base_link_Chasis -> base_link
- joint joint_2_Arm: parent base_link_Chasis -> base_link
- joint joint_front_left: parent base_link_Chasis -> base_link
- joint joint_front_right: parent base_link_Chasis -> base_link
- joint joint_rear_left: parent base_link_Chasis -> base_link
- joint joint_rear_right: parent base_link_Chasis -> base_link
- joint rgbd_link: parent base_link_Chasis -> base_link

Commit message: integration_launch

File: Ensamble_URDF_2ndT/urdf/Ensamble_URDF_2ndT.urdf (robot description, URDF)
Before this commit: robot robot, 12 links, 11 joints
Links:
- added link base_arm
Joints:
- added joint dummy_joint: type fixed, parent base_arm, child base_link
- joint joint_2_Arm: parent base_link -> base_arm

Commit message: Kalman tunning

File: Ensamble_URDF_2ndT/urdf/Ensamble_URDF_2ndT.urdf (robot description, URDF)
Before this commit: robot robot, 10 links, 9 joints
Links:
- removed link Link_1_1_wheel
- removed link Link_1_2_wheel
- removed link Link_1_3_wheel
- removed link Link_1_4_wheel
- removed link base_link_Chasis
- removed link map
- added link base_arm
- added link base_link, mass 15.1498884920758; collision mesh filename=package://ensamble_mobile/meshes/base_link_Chasis.STL; visual mesh filename=package://ensamble_mobile/meshes/base_link_Chasis.STL
- added link front_left_wheel, mass 0.622419475189309; collision mesh filename=package://ensamble_mobile/meshes/Link_1_4_wheel.STL; visual mesh filename=package://ensamble_mobile/meshes/Link_1_4_wheel.STL
- added link front_right_wheel, mass 0.622419475189309; collision mesh filename=package://ensamble_mobile/meshes/Link_1_3_wheel.STL; visual mesh filename=package://ensamble_mobile/meshes/Link_1_3_wheel.STL
- added link imu_link
- added link optical
- added link rear_left_wheel, mass 0.622419475189309; collision mesh filename=package://ensamble_mobile/meshes/Link_1_2_wheel.STL; visual mesh filename=package://ensamble_mobile/meshes/Link_1_2_wheel.STL
- added link rear_right_wheel, mass 0.622419475189312; collision mesh filename=package://ensamble_mobile/meshes/Link_1_1_wheel.STL; visual mesh filename=package://ensamble_mobile/meshes/Link_1_1_wheel.STL
- added link rgbd_cam, mass 0.1; visual box size=0.01 0.01 0.01
Joints:
- removed joint joint_1_1_wheel
- removed joint joint_1_2_wheel
- removed joint joint_1_3_wheel
- removed joint joint_1_4_wheel
- added joint imu_joint: type fixed, parent base_link, child imu_link, origin xyz=0.221 0.0 0.045 rpy=0.0 0.0 0.0
- added joint joint_front_left: type continuous, parent base_link, child front_left_wheel, origin xyz=0.08 0.19608 0.0195 rpy=-1.5708 0 0, axis 0 0 1
- added joint joint_front_right: type continuous, parent base_link, child front_right_wheel, origin xyz=0.08 -0.19478 0.0195 rpy=1.5708 0 0, axis 0 0 -1
- added joint joint_rear_left: type continuous, parent base_link, child rear_left_wheel, origin xyz=-0.12 0.19608 0.0195 rpy=-1.5708 0 0, axis 0 0 1
- added joint joint_rear_right: type continuous, parent base_link, child rear_right_wheel, origin xyz=-0.12 -0.19478 0.0195 rpy=1.5708 0 0, axis 0 0 -1
- added joint optical_joint: type fixed, parent rgbd_cam, child optical, origin xyz=0.0 0.0 0.0 rpy=-1.5708 0.0 -1.5708
- added joint rgbd_link: type fixed, parent base_link, child rgbd_cam, origin xyz=0.221 0.0 0.045 rpy=0.0 0.0 0.0
- joint dummy_joint: child base_link_Chasis -> base_link; parent map -> base_arm
- joint joint_2_Arm: parent base_link_Chasis -> base_link
- joint joint_3_Arm: limit lower=-0.6 upper=1.4 effort=100 velocity=100 -> lower=-1.6 upper=1.4 effort=100 velocity=100
- joint joint_4_Arm: limit lower=-1.57 upper=1.2 effort=100 velocity=100 -> lower=-1.87 upper=1.2 effort=100 velocity=100
- joint joint_5_Arm: limit lower=-2.8 upper=2.8 effort=100 velocity=100 -> lower=-2.5 upper=2.5 effort=100 velocity=100
