Commit message: Change rgbd reference

File: mobile/ensamble_mobile/urdf/mobile.urdf (robot description, URDF)
Before this commit: robot robot, 6 links, 5 joints
Links:
- added link rgbd_cam, mass 0.1; visual box size=0.01 0.01 0.01
- link base_link_Chasis: mass 5.34447797641956 -> 5.1498884920758
- link front_left_wheel: mass 0.622419475189308 -> 0.622419475189309
- link front_right_wheel: mass 0.622419475189312 -> 0.622419475189309
- link rear_left_wheel: mass 0.62241947518931 -> 0.622419475189309
- link rear_right_wheel: mass 0.62241947518931 -> 0.622419475189312
Joints:
- added joint rgbd_link: type fixed, parent base_link_Chasis, child rgbd_cam, origin xyz=0.0221 0.0 0.0045 rpy=0.0 0.0 0.0
- joint joint_front_right: origin xyz=0.0800000000000007 -0.133475850714851 0.0195000000000001 rpy=1.5707963267949 0 0 -> xyz=0.08 -0.19478 0.0195 rpy=1.5708 0 0
- joint joint_rear_left: origin xyz=-0.12 0.196084149285149 0.019499999999999 rpy=-1.5707963267949 0 0 -> xyz=-0.12 0.19608 0.0195 rpy=-1.5708 0 0
- joint joint_rear_right: origin xyz=-0.12 -0.13348 0.0195 rpy=1.5708 0 0 -> xyz=-0.12 -0.19478 0.0195 rpy=1.5708 0 0

Commit message: rgbd working

File: mobile/ensamble_mobile/urdf/mobile.urdf (robot description, URDF)
Before this commit: robot robot, 7 links, 6 joints
Links:
- added link optical
Joints:
- added joint optical_joint: type fixed, parent rgbd_cam, child optical, origin xyz=0.0 0.0 0.0 rpy=-1.5708 0.0 -1.5708
- joint rgbd_link: origin xyz=0.0221 0.0 0.0045 rpy=0.0 0.0 0.0 -> xyz=0.221 0.0 0.045 rpy=0.0 0.0 0.0

Commit message: Pal test

File: mobile/ensamble_mobile/urdf/mobile.urdf (robot description, URDF)
Before this commit: robot robot, 8 links, 7 joints
Links:
- added link Link_2_Arm, mass 0.628890750175801; collision mesh filename=package://Ensamble_URDF_2ndT/meshes/Link_2_Arm.STL; visual mesh filename=package://Ensamble_URDF_2ndT/meshes/Link_2_Arm.STL
- added link Link_3_Arm, mass 0.253359108687758; collision mesh filename=package://Ensamble_URDF_2ndT/meshes/Link_3_Arm.STL; visual mesh filename=package://Ensamble_URDF_2ndT/meshes/Link_3_Arm.STL
- added link Link_4_Arm, mass 0.5315; collision mesh filename=package://Ensamble_URDF_2ndT/meshes/Link_4_Arm.STL; visual mesh filename=package://Ensamble_URDF_2ndT/meshes/Link_4_Arm.STL
- added link Link_5_Arm, mass 0.34582; collision mesh filename=package://Ensamble_URDF_2ndT/meshes/Link_5_Arm.STL; visual mesh filename=package://Ensamble_URDF_2ndT/meshes/Link_5_Arm.STL
Joints:
- added joint joint_2_Arm: type revolute, parent base_link_Chasis, child Link_2_Arm, origin xyz=0 0 0.098503 rpy=0 0 0, axis 0 0 1, limit lower=-3.14 upper=3.14 effort=100 velocity=100
- added joint joint_3_Arm: type revolute, parent Link_2_Arm, child Link_3_Arm, origin xyz=0.063383 0.0021739 0.12369 rpy=1.5708 0 0, axis 0.034278 0 0.99941, limit lower=-0.6 upper=1.4 effort=100 velocity=100
- added joint joint_4_Arm: type revolute, parent Link_3_Arm, child Link_4_Arm, origin xyz=0.060241 0.1907 -0.0020662 rpy=0 0 0, axis -0.034278 0 -0.99941, limit lower=-1.57 upper=1.2 effort=100 velocity=100
- added joint joint_5_Arm: type revolute, parent Link_4_Arm, child Link_5_Arm, origin xyz=0.21278 -0.0095961 -0.0037813 rpy=0 0 0, axis -0.034278 0 -0.99941, limit lower=-2.8 upper=2.8 effort=100 velocity=100

Commit message: Adjusted_base_mass

File: mobile/ensamble_mobile/urdf/mobile.urdf (robot description, URDF)
Before this commit: robot robot, 12 links, 11 joints
Links:
- link base_link_Chasis: mass 5.1498884920758 -> 15.1498884920758

Commit message: Interneeeeeeeeeet

File: mobile/ensamble_mobile/urdf/mobile.urdf (robot description, URDF)
Before this commit: robot robot, 12 links, 11 joints
Links:
- removed link map
Joints:
- removed joint dummy_joint

Commit message: Fixed perception first ekf

File: mobile/ensamble_mobile/urdf/mobile.urdf (robot description, URDF)
Before this commit: robot robot, 11 links, 10 joints
Links:
- removed link base_link_Chasis
- added link base_link, mass 15.1498884920758; collision mesh filename=package://ensamble_mobile/meshes/base_link_Chasis.STL; visual mesh filename=package://ensamble_mobile/meshes/base_link_Chasis.STL
- added link imu_link
- added link map
Joints:
- added joint dummy_joint: type fixed, parent map, child base_link
- added joint imu_joint: type fixed, parent base_link, child imu_link, origin xyz=0.221 0.0 0.045 rpy=0.0 0.0 0.0
- joint joint_2_Arm: parent base_link_Chasis -> base_link
- joint joint_front_left: parent base_link_Chasis -> base_link
- joint joint_front_right: parent base_link_Chasis -> base_link
- joint joint_rear_left: parent base_link_Chasis -> base_link
- joint joint_rear_right: parent base_link_Chasis -> base_link
- joint rgbd_link: parent base_link_Chasis -> base_link

Commit message: integration_1

File: mobile/ensamble_mobile/urdf/mobile.urdf (robot description, URDF)
Before this commit: robot robot, 12 links, 11 joints
Links:
- removed link base_link_Chasis
- removed link map
- added link base_link, mass 15.1498884920758; collision mesh filename=package://ensamble_mobile/meshes/base_link_Chasis.STL; visual mesh filename=package://ensamble_mobile/meshes/base_link_Chasis.STL
- added link imu_link
Joints:
- removed joint dummy_joint
- added joint imu_joint: type fixed, parent base_link, child imu_link, origin xyz=0.221 0.0 0.045 rpy=0.0 0.0 0.0
- joint joint_2_Arm: parent base_link_Chasis -> base_link
- joint joint_front_left: parent base_link_Chasis -> base_link
- joint joint_front_right: parent base_link_Chasis -> base_link
- joint joint_rear_left: parent base_link_Chasis -> base_link
- joint joint_rear_right: parent base_link_Chasis -> base_link
- joint rgbd_link: parent base_link_Chasis -> base_link
